File: electronics/PSU Board/pi-tranceiver-psu/pi-tranceiver-psu.kicad_sch (KiCad schematic)
At the start: 67 parts, among them IC1 LTC4368IMS-2#PBF, IC2 LM2679S-ADJ_NOPB, J1 Phoenix PT2,5, J10 JST 01x04, J11 JST 01x04, J12 JST 01x02, J13 JST 01x02, J14 Phoenix PT2,5, J2 Phoenix PT2,5, J3 Phoenix PT2,5, J4 Phoenix PT2,5, J5 Phoenix PT2,5, J6 Phoenix PT2,5, J7 JST 01x02, J8 JST 01x02, J9 JST 01x02, Q1 DMT6002LPS-13, Q2 DMT6002LPS-13, Q3 Q_PMOS_GDS, Q4 BC547, Q5 BC547, Q6 BC547, SW1 SW_Push, U1 AMS1117-5.0, U2 AMS1117-5.0

Commit message: Update pi-tranceiver-psu.kicad_sch
Parts:
- added R18: 300R, symbol Device:R_Trim
- R12: value 3K24 -> 3K16
Connections:
- net at R12.2: now also R18.1; no longer JP1.1 (A)
- new net: JP1.1 (A), R18.2
Other:
- moved on the sheet: JP1, R15
Changed lines of the file:
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@@
   (junction (at 137.16 130.81) (diameter 0) (color 0 0 0 0)
   )
+  (junction (at 170.18 149.86) (diameter 0) (color 0 0 0 0)
+  )
   (junction (at 86.36 38.1) (diameter 0) (color 0 0 0 0)
   )
@@
   (junction (at 217.17 85.09) (diameter 0) (color 0 0 0 0)
   )
-  (junction (at 212.09 119.38) (diameter 0) (color 0 0 0 0)
-  )
   (junction (at 227.33 36.83) (diameter 0) (color 0 0 0 0)
   )
@@
   (junction (at 138.43 85.09) (diameter 0) (color 0 0 0 0)
   )
-  (junction (at 184.15 149.86) (diameter 0) (color 0 0 0 0)
-  )
   (junction (at 114.3 116.84) (diameter 0) (color 0 0 0 0)
   )
@@
   (junction (at 170.18 102.87) (diameter 0) (color 0 0 0 0)
   )
+  (junction (at 114.3 134.62) (diameter 0) (color 0 0 0 0)
+  )
   (junction (at 107.95 85.09) (diameter 0) (color 0 0 0 0)
   )
@@
   (junction (at 137.16 119.38) (diameter 0) (color 0 0 0 0)
   )
+  (junction (at 212.09 118.11) (diameter 0) (color 0 0 0 0)
+  )
   (junction (at 123.19 92.71) (diameter 0) (color 0 0 0 0)
   )
@@
   (junction (at 81.28 85.09) (diameter 0) (color 0 0 0 0)
   )
-  (junction (at 114.3 134.62) (diameter 0) (color 0 0 0 0)
-  )
   (junction (at 184.15 33.02) (diameter 0) (color 0 0 0 0)
   )
@@
     (stroke (width 0) (type default) (color 0 0 0 0))
   )
-  (wire (pts (xy 114.3 138.43) (xy 114.3 134.62))
-    (stroke (width 0) (type default) (color 0 0 0 0))
-  )
   (wire (pts (xy 190.5 67.31) (xy 190.5 60.96))
     (stroke (width 0) (type default) (color 0 0 0 0))
@@
     (stroke (width 0) (type default) (color 0 0 0 0))
   )
-  (wire (pts (xy 163.83 119.38) (xy 212.09 119.38))
-    (stroke (width 0) (type default) (color 0 0 0 0))
-  )
   (wire (pts (xy 78.74 114.3) (xy 97.79 114.3))
     (stroke (width 0) (type default) (color 0 0 0 0))
@@
     (stroke (width 0) (type default) (color 0 0 0 0))
   )
+  (wire (pts (xy 163.83 125.73) (xy 196.85 125.73))
+    (stroke (width 0) (type default) (color 0 0 0 0))
+  )
   (wire (pts (xy 220.98 132.08) (xy 226.06 132.08))
     (stroke (width 0) (type default) (color 0 0 0 0))
@@
     (stroke (width 0) (type default) (color 0 0 0 0))
   )
+  (wire (pts (xy 196.85 125.73) (xy 196.85 118.11))
+    (stroke (width 0) (type default) (color 0 0 0 0))
+  )
   (wire (pts (xy 250.19 81.28) (xy 247.65 81.28))
     (stroke (width 0) (type default) (color 0 0 0 0))
@@
     (stroke (width 0) (type default) (color 0 0 0 0))
   )
+  (wire (pts (xy 170.18 111.76) (xy 170.18 114.3))
+    (stroke (width 0) (type default) (color 0 0 0 0))
+  )
   (wire (pts (xy 144.78 102.87) (xy 157.48 102.87))
     (stroke (width 0) (type default) (color 0 0 0 0))
@@
     (stroke (width 0) (type default) (color 0 0 0 0))
   )
-  (wire (pts (xy 212.09 115.57) (xy 212.09 119.38))
-    (stroke (width 0) (type default) (color 0 0 0 0))
-  )
   (wire (pts (xy 157.48 102.87) (xy 170.18 102.87))
     (stroke (width 0) (type default) (color 0 0 0 0))
@@
     (stroke (width 0) (type default) (color 0 0 0 0))
   )
+  (wire (pts (xy 196.85 118.11) (xy 212.09 118.11))
+    (stroke (width 0) (type default) (color 0 0 0 0))
+  )
   (wire (pts (xy 81.28 57.15) (xy 81.28 59.69))
     (stroke (width 0) (type default) (color 0 0 0 0))
@@
     (stroke (width 0) (type default) (color 0 0 0 0))
   )
-  (wire (pts (xy 157.48 111.76) (xy 157.48 123.19))
+  (wire (pts (xy 157.48 111.76) (xy 157.48 129.54))
+    (stroke (width 0) (type default) (color 0 0 0 0))
+  )
+  (wire (pts (xy 114.3 134.62) (xy 114.3 142.24))
     (stroke (width 0) (type default) (color 0 0 0 0))
   )
@@
     (stroke (width 0) (type default) (color 0 0 0 0))
   )
-  (wire (pts (xy 184.15 138.43) (xy 114.3 138.43))
-    (stroke (width 0) (type default) (color 0 0 0 0))
-  )
   (wire (pts (xy 109.22 105.41) (xy 114.3 105.41))
     (stroke (width 0) (type default) (color 0 0 0 0))
@@
     (stroke (width 0) (type default) (color 0 0 0 0))
   )
-  (wire (pts (xy 184.15 148.59) (xy 184.15 149.86))
+  (wire (pts (xy 114.3 149.86) (xy 170.18 149.86))
     (stroke (width 0) (type default) (color 0 0 0 0))
   )
@@
     (stroke (width 0) (type default) (color 0 0 0 0))
   )
-  (wire (pts (xy 170.18 111.76) (xy 170.18 123.19))
-    (stroke (width 0) (type default) (color 0 0 0 0))
-  )
   (wire (pts (xy 199.39 153.67) (xy 199.39 156.21))
     (stroke (width 0) (type default) (color 0 0 0 0))
@@
     (stroke (width 0) (type default) (color 0 0 0 0))
   )
+  (wire (pts (xy 212.09 118.11) (xy 212.09 120.65))
+    (stroke (width 0) (type default) (color 0 0 0 0))
+  )
   (wire (pts (xy 66.04 85.09) (xy 73.66 85.09))
     (stroke (width 0) (type default) (color 0 0 0 0))
@@
     (stroke (width 0) (type default) (color 0 0 0 0))
   )
+  (wire (pts (xy 170.18 121.92) (xy 170.18 129.54))
+    (stroke (width 0) (type default) (color 0 0 0 0))
+  )
   (wire (pts (xy 130.81 50.8) (xy 157.48 50.8))
     (stroke (width 0) (type default) (color 0 0 0 0))
@@
     (stroke (width 0) (type default) (color 0 0 0 0))
   )
-  (wire (pts (xy 212.09 119.38) (xy 212.09 120.65))
+  (wire (pts (xy 212.09 115.57) (xy 212.09 118.11))
     (stroke (width 0) (type default) (color 0 0 0 0))
   )
@@
   )
   (wire (pts (xy 40.64 60.96) (xy 40.64 50.8))
-    (stroke (width 0) (type default) (color 0 0 0 0))
-  )
-  (wire (pts (xy 184.15 140.97) (xy 184.15 138.43))
     (stroke (width 0) (type default) (color 0 0 0 0))
   )
@@
     (pin "2")
   )
+  (symbol (lib_id "Device:R_Trim") (at 170.18 118.11 0) (unit 1)
+    (in_bom yes) (on_board yes) (fields_autoplaced)
+    (property "Reference" "R18" (id 0) (at 173.99 116.8399 0)
+      (effects (font (size 1.27 1.27)) (justify left))
+    )
+    (property "Value" "300R" (id 1) (at 173.99 119.3799 0)
+      (effects (font (size 1.27 1.27)) (justify left))
+    )
+    (property "Footprint" "" (id 2) (at 168.402 118.11 90)
+      (effects (font (size 1.27 1.27)) hide)
+    )
+    (property "Datasheet" "~" (id 3) (at 170.18 118.11 0)
+      (effects (font (size 1.27 1.27)) hide)
+    )
+    (pin "1")
+    (pin "2")
+  )
   (symbol (lib_id "Connector:Screw_Terminal_01x02") (at 247.65 30.48 0) (unit 1)
     (in_bom yes) (on_board yes) (fields_autoplaced)
@@
     (pin "2")
   )
-  (symbol (lib_id "Jumper:Jumper_3_Bridged12") (at 163.83 123.19 180) (unit 1)
-    (in_bom yes) (on_board yes) (fields_autoplaced)
-    (property "Reference" "JP1" (id 0) (at 163.83 127 0))
-    (property "Value" "5.1V / 8.4V" (id 1) (at 163.83 129.54 0))
-    (property "Footprint" "" (id 2) (at 163.83 123.19 0)
-      (effects (font (size 1.27 1.27)) hide)
-    )
-    (property "Datasheet" "~" (id 3) (at 163.83 123.19 0)
+  (symbol (lib_id "Jumper:Jumper_3_Bridged12") (at 163.83 129.54 180) (unit 1)
+    (in_bom yes) (on_board yes) (fields_autoplaced)
+    (property "Reference" "JP1" (id 0) (at 163.83 133.35 0))
+    (property "Value" "5.1V / 8.4V" (id 1) (at 163.83 135.89 0))
+    (property "Footprint" "" (id 2) (at 163.83 129.54 0)
+      (effects (font (size 1.27 1.27)) hide)
+    )
+    (property "Datasheet" "~" (id 3) (at 163.83 129.54 0)
       (effects (font (size 1.27 1.27)) hide)
     )
@@
     (pin "2")
   )
-  (symbol (lib_id "Device:R") (at 184.15 144.78 0) (unit 1)
-    (in_bom yes) (on_board yes)
-    (property "Reference" "R15" (id 0) (at 185.928 143.6116 0)
-      (effects (font (size 1.27 1.27)) (justify left))
-    )
-    (property "Value" "100K" (id 1) (at 185.928 145.923 0)
-      (effects (font (size 1.27 1.27)) (justify left))
-    )
-    (property "Footprint" "Resistor_SMD:R_0805_2012Metric_Pad1.20x1.40mm_HandSolder" (id 2) (at 182.372 144.78 90)
-      (effects (font (size 1.27 1.27)) hide)
-    )
-    (property "Datasheet" "~" (id 3) (at 184.15 144.78 0)
+  (symbol (lib_id "Device:R") (at 114.3 146.05 0) (unit 1)
+    (in_bom yes) (on_board yes)
+    (property "Reference" "R15" (id 0) (at 116.078 144.8816 0)
+      (effects (font (size 1.27 1.27)) (justify left))
+    )
+    (property "Value" "100K" (id 1) (at 116.078 147.193 0)
+      (effects (font (size 1.27 1.27)) (justify left))
+    )
+    (property "Footprint" "Resistor_SMD:R_0805_2012Metric_Pad1.20x1.40mm_HandSolder" (id 2) (at 112.522 146.05 90)
+      (effects (font (size 1.27 1.27)) hide)
+    )
+    (property "Datasheet" "~" (id 3) (at 114.3 146.05 0)
       (effects (font (size 1.27 1.27)) hide)
     )
@@
       (effects (font (size 1.27 1.27)) (justify left))
     )
-    (property "Value" "3K24" (id 1) (at 171.958 109.093 0)
+    (property "Value" "3K16" (id 1) (at 171.958 109.093 0)
       (effects (font (size 1.27 1.27)) (justify left))
     )
@@
     )
     (path "/857a622e-ee63-427d-91b0-51b3917a95d8"
-      (reference "R12") (unit 1) (value "3K24") (footprint "Resistor_SMD:R_0805_2012Metric_Pad1.20x1.40mm_HandSolder")
+      (reference "R12") (unit 1) (value "3K16") (footprint "Resistor_SMD:R_0805_2012Metric_Pad1.20x1.40mm_HandSolder")
     )
     (path "/3b9eba01-bacc-48e0-b11d-1d7b67e62764"
@@
       (reference "R17") (unit 1) (value "100K") (footprint "Resistor_SMD:R_0805_2012Metric_Pad1.20x1.40mm_HandSolder")
     )
+    (path "/1baebc0d-31bb-48b8-adf8-ab0e95501414"
+      (reference "R18") (unit 1) (value "300R") (footprint "")
+    )
     (path "/f0392e65-5f42-4db7-bc59-f587f1892960"
