File: electronics/PSU Board/pi-tranceiver-psu/pi-tranceiver-psu.kicad_sch (KiCad schematic)
At the start: 68 parts, among them IC1 LTC4368IMS-2#PBF, IC2 LM2679S-ADJ_NOPB, J1 Phoenix PT2,5, J10 JST 01x04, J11 JST 01x04, J12 JST 01x02, J13 JST 01x02, J14 Phoenix PT2,5, J2 Phoenix PT2,5, J3 Phoenix PT2,5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

Commit message: Update pi-tranceiver-psu.kicad_sch
Other:
- note added: "ovp"
Changed lines of the file:
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@@
+    (effects (font (size 1.27 1.27)) (justify left bottom))
+  )
+  (text "ovp" (at 100.33 134.62 0)
     (effects (font (size 1.27 1.27)) (justify left bottom))
   )
