File: electronics/pi_transceiver_hat/pi_transceiver_hat.kicad_sch (KiCad schematic)
At the start: 40 parts, among them J1 Raspberry_Pi_2_3, J10 +5v Power, J11 i2c, J12 i2c, J13 i2c, J14 i2c, J15 Meter, J2 GND, J3 RX Board, J4 1 wire, J5 PSU Board, J6 +5V, J7 UART, J8 +3.3V, J9 PA Board, M1 Fan 1, M2 Fan 2, Q1 2N7000, Q2 2N7000, U1 MCP4725xxx-xCH

Commit message: Hat PCB alpha design
Parts:
- C1: footprint Capacitor_SMD:CP_Elec_10x12.6 -> Capacitor_SMD:CP_Elec_4x5.4
- C3, C4, C5: value C -> 100nF
Changed lines of the file:
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@@
   )
   (symbol (lib_id "power:+3V3") (at 91.44 53.34 0) (unit 1)
-    (in_bom yes) (on_board yes) (fields_autoplaced)
+    (in_bom yes) (on_board yes)
     (property "Reference" "#PWR029" (id 0) (at 91.44 57.15 0)
       (effects (font (size 1.27 1.27)) hide)
     )
-    (property "Value" "+3V3" (id 1) (at 91.44 49.7355 0))
+    (property "Value" "+3V3" (id 1) (at 88.646 50.546 0))
     (property "Footprint" "" (id 2) (at 91.44 53.34 0)
       (effects (font (size 1.27 1.27)) hide)
@@
   )
   (symbol (lib_id "Device:C") (at 114.046 43.942 180) (unit 1)
-    (in_bom yes) (on_board yes) (fields_autoplaced)
-    (property "Reference" "C4" (id 0) (at 116.967 43.0335 0)
+    (in_bom yes) (on_board yes)
+    (property "Reference" "C4" (id 0) (at 107.95 39.37 0)
       (effects (font (size 1.27 1.27)) (justify right))
     )
-    (property "Value" "C" (id 1) (at 116.967 45.8086 0)
+    (property "Value" "100nF" (id 1) (at 107.188 41.656 0)
       (effects (font (size 1.27 1.27)) (justify right))
     )
@@
   )
   (symbol (lib_id "power:+5V") (at 83.82 53.34 0) (unit 1)
-    (in_bom yes) (on_board yes) (fields_autoplaced)
+    (in_bom yes) (on_board yes)
     (property "Reference" "#PWR023" (id 0) (at 83.82 57.15 0)
       (effects (font (size 1.27 1.27)) hide)
     )
-    (property "Value" "+5V" (id 1) (at 83.82 49.7355 0))
+    (property "Value" "+5V" (id 1) (at 80.264 51.308 0))
     (property "Footprint" "" (id 2) (at 83.82 53.34 0)
       (effects (font (size 1.27 1.27)) hide)
@@
   )
   (symbol (lib_id "power:+5V") (at 86.36 53.34 0) (unit 1)
-    (in_bom yes) (on_board yes) (fields_autoplaced)
+    (in_bom yes) (on_board yes)
     (property "Reference" "#PWR026" (id 0) (at 86.36 57.15 0)
       (effects (font (size 1.27 1.27)) hide)
     )
-    (property "Value" "+5V" (id 1) (at 86.36 49.7355 0))
+    (property "Value" "+5V" (id 1) (at 85.344 48.768 0))
     (property "Footprint" "" (id 2) (at 86.36 53.34 0)
       (effects (font (size 1.27 1.27)) hide)
@@
     (in_bom yes) (on_board yes) (fields_autoplaced)
     (property "Reference" "C5" (id 0) (at 149.86 45.6905 90))
-    (property "Value" "C" (id 1) (at 149.86 48.4656 90))
+    (property "Value" "100nF" (id 1) (at 149.86 48.4656 90))
     (property "Footprint" "Capacitor_SMD:C_0805_2012Metric_Pad1.18x1.45mm_HandSolder" (id 2) (at 153.67 50.8508 0)
       (effects (font (size 1.27 1.27)) hide)
@@
       (effects (font (size 1.27 1.27)) (justify right))
     )
-    (property "Footprint" "Capacitor_SMD:CP_Elec_10x12.6" (id 2) (at 29.5148 38.1 0)
+    (property "Footprint" "Capacitor_SMD:CP_Elec_4x5.4" (id 2) (at 29.5148 38.1 0)
       (effects (font (size 1.27 1.27)) hide)
     )
@@
   )
   (symbol (lib_id "power:GND") (at 104.14 51.308 270) (unit 1)
-    (in_bom yes) (on_board yes) (fields_autoplaced)
+    (in_bom yes) (on_board yes)
     (property "Reference" "#PWR066" (id 0) (at 97.79 51.308 0)
       (effects (font (size 1.27 1.27)) hide)
     )
-    (property "Value" "GND" (id 1) (at 100.9651 51.787 90)
+    (property "Value" "GND" (id 1) (at 106.934 52.578 90)
       (effects (font (size 1.27 1.27)) (justify right))
     )
@@
   (symbol (lib_id "Connector:Raspberry_Pi_2_3") (at 88.9 86.36 0) (unit 1)
     (in_bom yes) (on_board yes)
-    (property "Reference" "J1" (id 0) (at 96.012 51.816 0)
-      (effects (font (size 1.27 1.27)) (justify left))
-    )
-    (property "Value" "Raspberry_Pi_2_3" (id 1) (at 96.012 54.61 0)
+    (property "Reference" "J1" (id 0) (at 70.866 51.054 0)
+      (effects (font (size 1.27 1.27)) (justify left))
+    )
+    (property "Value" "Raspberry_Pi_2_3" (id 1) (at 64.516 53.848 0)
       (effects (font (size 1.27 1.27)) (justify left))
     )
@@
   )
   (symbol (lib_id "power:GND") (at 114.046 47.752 0) (unit 1)
-    (in_bom yes) (on_board yes) (fields_autoplaced)
+    (in_bom yes) (on_board yes)
     (property "Reference" "#PWR068" (id 0) (at 114.046 54.102 0)
       (effects (font (size 1.27 1.27)) hide)
     )
-    (property "Value" "GND" (id 1) (at 114.046 52.3145 0))
+    (property "Value" "GND" (id 1) (at 118.11 50.546 0))
     (property "Footprint" "" (id 2) (at 114.046 47.752 0)
       (effects (font (size 1.27 1.27)) hide)
@@
   )
   (symbol (lib_id "Device:C") (at 104.14 47.498 180) (unit 1)
-    (in_bom yes) (on_board yes) (fields_autoplaced)
-    (property "Reference" "C3" (id 0) (at 107.061 46.5895 0)
+    (in_bom yes) (on_board yes)
+    (property "Reference" "C3" (id 0) (at 98.044 48.006 0)
       (effects (font (size 1.27 1.27)) (justify right))
     )
-    (property "Value" "C" (id 1) (at 107.061 49.3646 0)
+    (property "Value" "100nF" (id 1) (at 94.742 45.72 0)
       (effects (font (size 1.27 1.27)) (justify right))
     )
@@
     )
     (path "/85de51b3-51fb-4e03-b355-02879d9e4d94"
-      (reference "C1") (unit 1) (value "10uF") (footprint "Capacitor_SMD:CP_Elec_10x12.6")
+      (reference "C1") (unit 1) (value "10uF") (footprint "Capacitor_SMD:CP_Elec_4x5.4")
     )
     (path "/d462c439-0fc3-490f-b4b6-390c514f4af3"
@@
     )
     (path "/cc8065a2-6f18-4933-ac1b-69d166dc3a05"
-      (reference "C3") (unit 1) (value "C") (footprint "Capacitor_SMD:C_0805_2012Metric_Pad1.18x1.45mm_HandSolder")
+      (reference "C3") (unit 1) (value "100nF") (footprint "Capacitor_SMD:C_0805_2012Metric_Pad1.18x1.45mm_HandSolder")
     )
     (path "/1fd42365-82fc-4428-b579-9578c263211e"
-      (reference "C4") (unit 1) (value "C") (footprint "Capacitor_SMD:C_0805_2012Metric_Pad1.18x1.45mm_HandSolder")
+      (reference "C4") (unit 1) (value "100nF") (footprint "Capacitor_SMD:C_0805_2012Metric_Pad1.18x1.45mm_HandSolder")
     )
     (path "/53316fe2-cc5c-4ac6-81f1-37cee80131b6"
-      (reference "C5") (unit 1) (value "C") (footprint "Capacitor_SMD:C_0805_2012Metric_Pad1.18x1.45mm_HandSolder")
+      (reference "C5") (unit 1) (value "100nF") (footprint "Capacitor_SMD:C_0805_2012Metric_Pad1.18x1.45mm_HandSolder")
     )
     (path "/4ab3d9f5-b837-473c-9443-6634e8fba6c1"
