File: electronics/PA_Board/PA_Protection.kicad_sch (KiCad schematic)
At the start: 53 parts, among them J1 USB_B_Micro, J2 Conn_01x05, J3 Conn_01x05, J4 Conn_01x04, SW1 SW_Push, U1 ATSAMD21E18A-A, U2 LM75B, U3 LM2904

Commit message: PCB updates and gerbers
Parts:
- D2: footprint LED_SMD:LED-APA102-2020 -> Pi_Tx:LED-APA102-2020
- U2, U3: footprint Package_SO:SO-8_3.9x4.9mm_P1.27mm -> Package_SO:SOIC-8_3.9x4.9mm_P1.27mm
Changed lines of the file:
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@@
     (property "Reference" "U3" (id 0) (at 234.95 25.5102 0))
     (property "Value" "LM2904" (id 1) (at 234.95 28.0471 0))
-    (property "Footprint" "Package_SO:SO-8_3.9x4.9mm_P1.27mm" (id 2) (at 234.95 34.29 0)
+    (property "Footprint" "Package_SO:SOIC-8_3.9x4.9mm_P1.27mm" (id 2) (at 234.95 34.29 0)
       (effects (font (size 1.27 1.27)) hide)
     )
@@
       (effects (font (size 1.27 1.27)) (justify left))
     )
-    (property "Footprint" "LED_SMD:LED-APA102-2020" (id 2) (at 116.205 67.945 0)
+    (property "Footprint" "Pi_Tx:LED-APA102-2020" (id 2) (at 116.205 67.945 0)
       (effects (font (size 1.27 1.27)) (justify left top) hide)
     )
@@
     (property "Reference" "U3" (id 0) (at 234.95 67.4202 0))
     (property "Value" "LM2904" (id 1) (at 234.95 69.9571 0))
-    (property "Footprint" "Package_SO:SO-8_3.9x4.9mm_P1.27mm" (id 2) (at 234.95 76.2 0)
+    (property "Footprint" "Package_SO:SOIC-8_3.9x4.9mm_P1.27mm" (id 2) (at 234.95 76.2 0)
       (effects (font (size 1.27 1.27)) hide)
     )
@@
     (pin "1")
   )
-  (symbol (lib_id "Diode:1N914") (at 229.235 62.23 0) (unit 1)
+  (symbol (lib_name "1N914_1") (lib_id "Diode:1N914") (at 229.235 62.23 0) (unit 1)
     (in_bom yes) (on_board yes) (fields_autoplaced)
     (property "Reference" "D6" (id 0) (at 229.235 57.2602 0))
@@
       (effects (font (size 1.27 1.27)) (justify left))
     )
-    (property "Footprint" "Package_SO:SO-8_3.9x4.9mm_P1.27mm" (id 2) (at 166.37 60.96 0)
+    (property "Footprint" "Package_SO:SOIC-8_3.9x4.9mm_P1.27mm" (id 2) (at 166.37 60.96 0)
       (effects (font (size 1.27 1.27)) hide)
     )
@@
       (effects (font (size 1.27 1.27)) (justify left))
     )
-    (property "Footprint" "Package_SO:SO-8_3.9x4.9mm_P1.27mm" (id 2) (at 247.015 117.475 0)
-      (effects (font (size 1.27 1.27)) hide)
-    )
+    (property "Footprint" "Package_SO:SOIC-8_3.9x4.9mm_P1.27mm" (id 2) (at 247.015 117.475 0)
+      (effects (font (size 1.27 1.27)) hide)
+    )

Commit message: Update Kicad Schematic and PCB
Fixed: D8 was reversed, Q2 wrong footprint.
Some component values added or changed
Documentation added
Parts:
- R12: value 10k -> 47k
- R15: value 100k -> 10k
Other:
- note added: "Arduino Pin Mapping ATSAMD21E18 I/O Multiplexer 0 PA00 DOTSTAR SDI 1 PA01 DOTSTAR CLK 2 PA02 UNUSED GPIO 3 PA03 ADC_FWD 4 PA04 ADC_REV 5 PA05 ADC_Vgg 6 PA06 TX_Relay_Out 7 PA07 UNUSED 8 PA08 SERCOM0 PAD 0 SDA/TXD 9 PA09 SERCOM0 PAD 1 SCL/RX 10 PA10 Watchdog LED 11 PA11 SLAVE GPIO INT 12 PA14 UNUSED GPIO 13 PA15 En_Vgg_PA 14 PA16 SERCOM1 PAD 0 Ext_SDA 15 PA17 SERCOM1 PAD 1 Ext_SCL 16 PA18 USB Host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"
- moved on the sheet: C1, C2, C3, C4, C5, C6, D1, D2, D3, J1, J2, L1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

Commit message: Add PA Board tests
Add PA Board Arduino Tests
Parts:
- D3: value LED -> LED_Orange
- R22, R23: value 330 -> 330R
Changed lines of the file:
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@@
     (in_bom yes) (on_board yes) (fields_autoplaced)
     (property "Reference" "R22" (id 0) (at 250.19 68.9442 90))
-    (property "Value" "330" (id 1) (at 250.19 71.4811 90))
+    (property "Value" "330R" (id 1) (at 250.19 71.4811 90))
     (property "Footprint" "Resistor_SMD:R_0603_1608Metric" (id 2) (at 250.19 75.438 90)
       (effects (font (size 1.27 1.27)) hide)
@@
       (effects (font (size 1.27 1.27)) (justify right))
     )
-    (property "Value" "LED" (id 1) (at 128.651 90.9197 90)
+    (property "Value" "LED_Orange" (id 1) (at 128.651 90.9197 90)
       (effects (font (size 1.27 1.27)) (justify right))
     )
@@
     (in_bom yes) (on_board yes) (fields_autoplaced)
     (property "Reference" "R23" (id 0) (at 250.825 29.5742 90))
-    (property "Value" "330" (id 1) (at 250.825 32.1111 90))
+    (property "Value" "330R" (id 1) (at 250.825 32.1111 90))
     (property "Footprint" "Resistor_SMD:R_0603_1608Metric" (id 2) (at 250.825 36.068 90)
       (effects (font (size 1.27 1.27)) hide)

Commit message: Merge branch 'main' of https://github.com/M0LTE/pi-transceiver
Addition of PA Board version 2 Kicad files
Other:
- note added: "Arduino Pin Mapping ATSAMD21E18 I/O Multiplexer 0 PA00 DOTSTAR SDI 1 PA01 DOTSTAR CLK 2 PA03 ADC_FWD 3 PA04 ADC_REV 4 PA05 ADC_Vgg 5 PA06 TX_Relay_Out 6 PA08 SERCOM0 PAD 0 Slave_SDA 7 PA09 SERCOM0 PAD 1 Slave_SCL 8 PA10 Watchdog LED 9 PA11 SLAVE GPIO INT 10 PA15 En_Vgg_PA 11 PA16 SERCOM1 PAD 0 Ext_SDA 12 PA17 SERCOM1 PAD 1 Ext_SCL 13 PA19 LM75 Interrupt 14 PA22 SERCOM3 PAD 0 Int_SDA 15 PA23 SERCO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"
- note added: "Compensating RF Detector Buffer Amplifiers"
- note added: "I2C Address 0x48"
- note removed: "Arduino Pin Mapping ATSAMD21E18 I/O Multiplexer 0 PA00 DOTSTAR SDI 1 PA01 DOTSTAR CLK 2 PA02 UNUSED GPIO 3 PA03 ADC_FWD 4 PA04 ADC_REV 5 PA05 ADC_Vgg 6 PA06 TX_Relay_Out 7 PA07 UNUSED 8 PA08 SERCOM0 PAD 0 SDA/TXD 9 PA09 SERCOM0 PAD 1 SCL/RX 10 PA10 Watchdog LED 11 PA11 SLAVE GPIO INT 12 PA14 UNUSED GPIO 13 PA15 En_Vgg_PA 14 PA16 SERCOM1 PAD 0 Ext_SDA 15 PA17 SERCOM1 PAD 1 Ext_SCL 16 PA18 USB Host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"
- moved on the sheet: C10, U3C
