File: electronics/PA_Board/PA_RF.kicad_sch (KiCad schematic)
At the start: 64 parts, among them J6 Conn_Coaxial, J7 Conn_Coaxial, J8 Conn_Coaxial, J9 Conn_Coaxial, K1 G6E, Q2 BC848W, U10 RA35H1516M, U9 SPF5189Z

Commit message: PCB updates and gerbers
Parts:
- added U11: Directional_Coupler, Pi_Tx:Wiggly Coupler, symbol Pi_PA:Directional_Coupler
- L5, L7: footprint Inductor_SMD:L_Neosid_Air-Coil_SML_3turn_HDM0331A -> Pi_Tx:Wire_Inductor 12x8.5
- L6: footprint Inductor_SMD:L_Neosid_Air-Coil_SML_3turn_HDM0331A -> Pi_Tx:Wire_Inductor 15.5x8.5
Connections:
- net at C45.1, K1.12, L7.2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: now also U11.1 (RF)
- net at D12.2 (A), D13.1 (K), R44.2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: now also U11.2 (Fterm)
- net at D14.2 (A), D15.1 (K), R40.1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: now also U11.3 (Rterm)
- net VDD_GAIN renamed +5V
Other:
- note removed: "Directional Coupler"
- moved on the sheet: C38, C39, C40, C41, C42, C43, C44, C45, C47, C48, C51, D12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

Commit message: Update Kicad Schematic and PCB
Fixed: D8 was reversed, Q2 wrong footprint.
Some component values added or changed
Documentation added
Parts:
- C38: value C -> 9p1
- C39, C42: value C -> 18p
- C40, C43: value C -> NF
- C41: value C -> 3p
- C45: value C -> 6p8
- L5, L7: value L -> 34nH
- L6: value L -> 46nH
- Q2: footprint Package_TO_SOT_SMD:SOT-323_SC-70 -> Package_TO_SOT_SMD:SOT-23
Changed lines of the file:
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@@
       (effects (font (size 1.27 1.27)) (justify left))
     )
-    (property "Value" "C" (id 1) (at 157.861 110.9222 0)
+    (property "Value" "18p" (id 1) (at 150.495 112.395 0)
       (effects (font (size 1.27 1.27)) (justify left))
     )
@@
     (in_bom yes) (on_board yes)
     (property "Reference" "C38" (id 0) (at 130.81 91.44 90))
-    (property "Value" "C" (id 1) (at 130.81 98.425 90))
+    (property "Value" "9p1" (id 1) (at 133.985 98.425 90))
     (property "Footprint" "Inductor_SMD:L_1206_3216Metric" (id 2) (at 134.62 94.2848 0)
       (effects (font (size 1.27 1.27)) hide)
@@
       (effects (font (size 1.27 1.27)) (justify left))
     )
-    (property "Value" "C" (id 1) (at 163.576 110.9222 0)
+    (property "Value" "NF" (id 1) (at 161.29 111.76 0)
       (effects (font (size 1.27 1.27)) (justify left))
     )
@@
       (effects (font (size 1.27 1.27)) (justify left))
     )
-    (property "Footprint" "Package_TO_SOT_SMD:SOT-323_SC-70" (id 2) (at 268.605 146.05 0)
+    (property "Footprint" "Package_TO_SOT_SMD:SOT-23" (id 2) (at 268.605 146.05 0)
       (effects (font (size 1.27 1.27) italic) (justify left) hide)
     )
@@
       (effects (font (size 1.27 1.27)) (justify left))
     )
-    (property "Value" "C" (id 1) (at 145.796 110.9222 0)
+    (property "Value" "NF" (id 1) (at 143.51 111.76 0)
       (effects (font (size 1.27 1.27)) (justify left))
     )
@@
   )
   (symbol (lib_id "Device:C") (at 171.45 109.22 0) (unit 1)
-    (in_bom yes) (on_board yes) (fields_autoplaced)
+    (in_bom yes) (on_board yes)
     (property "Reference" "C45" (id 0) (at 174.371 108.3853 0)
       (effects (font (size 1.27 1.27)) (justify left))
     )
-    (property "Value" "C" (id 1) (at 174.371 110.9222 0)
+    (property "Value" "6p8" (id 1) (at 172.72 112.395 0)
       (effects (font (size 1.27 1.27)) (justify left))
     )
@@
     (in_bom yes) (on_board yes)
     (property "Reference" "L6" (id 0) (at 149.225 104.14 90))
-    (property "Value" "L" (id 1) (at 149.225 101.1991 90))
+    (property "Value" "46nH" (id 1) (at 149.225 101.1991 90))
     (property "Footprint" "Pi_Tx:Wire_Inductor 15.5x8.5" (id 2) (at 149.225 102.87 0)
       (effects (font (size 1.27 1.27)) hide)
@@
     (in_bom yes) (on_board yes)
     (property "Reference" "C41" (id 0) (at 149.225 91.44 90))
-    (property "Value" "C" (id 1) (at 149.225 98.425 90))
+    (property "Value" "3p" (id 1) (at 151.765 98.425 90))
     (property "Footprint" "Inductor_SMD:L_1206_3216Metric" (id 2) (at 153.035 94.2848 0)
       (effects (font (size 1.27 1.27)) hide)
@@
     (in_bom yes) (on_board yes)
     (property "Reference" "L5" (id 0) (at 130.81 104.14 90))
-    (property "Value" "L" (id 1) (at 130.81 101.1991 90))
+    (property "Value" "34nH" (id 1) (at 130.81 101.1991 90))
     (property "Footprint" "Pi_Tx:Wire_Inductor 12x8.5" (id 2) (at 130.81 102.87 0)
       (effects (font (size 1.27 1.27)) hide)
@@
     (in_bom yes) (on_board yes)
     (property "Reference" "L7" (id 0) (at 165.735 104.14 90))
-    (property "Value" "L" (id 1) (at 165.735 100.965 90))
+    (property "Value" "34nH" (id 1) (at 165.735 100.965 90))
     (property "Footprint" "Pi_Tx:Wire_Inductor 12x8.5" (id 2) (at 165.735 102.87 0)
       (effects (font (size 1.27 1.27)) hide)
@@
       (effects (font (size 1.27 1.27)) (justify left))
     )
-    (property "Value" "C" (id 1) (at 140.081 110.9222 0)
-      (effects (font (size 1.27 1.27)) (justify left))
-    )
+    (property "Value" "18p" (id 1) (at 132.715 112.395 0)
+      (effects (font (size 1.27 1.27)) (justify left))
+    )

Commit message: Add PA Board tests
Add PA Board Arduino Tests
Parts:
- D17: value LED -> LED_Red
- R37, R39, R40, R41, R44, R45: value 150 -> 150R
- R38: value 37.4 -> 37.4R
- R42: value 49.9 -> 49.9R
Changed lines of the file:
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@@
       (effects (font (size 1.27 1.27)) (justify right))
     )
-    (property "Value" "LED" (id 1) (at 280.035 134.62 90)
+    (property "Value" "LED_Red" (id 1) (at 270.51 125.095 90)
       (effects (font (size 1.27 1.27)) (justify right))
     )
@@
   )
   (symbol (lib_id "Device:L") (at 249.555 121.92 0) (unit 1)
-    (in_bom yes) (on_board yes) (fields_autoplaced)
-    (property "Reference" "L11" (id 0) (at 250.825 121.0853 0)
+    (in_bom yes) (on_board yes)
+    (property "Reference" "L11" (id 0) (at 245.745 120.65 0)
       (effects (font (size 1.27 1.27)) (justify left))
     )
@@
       (effects (font (size 1.27 1.27)) (justify left))
     )
-    (property "Value" "49.9" (id 1) (at 212.725 68.58 0)
+    (property "Value" "49.9R" (id 1) (at 212.725 68.58 0)
       (effects (font (size 1.27 1.27)) (justify left))
     )
@@
       (effects (font (size 1.27 1.27)) (justify left))
     )
-    (property "Value" "150" (id 1) (at 226.695 95.885 0)
+    (property "Value" "150R" (id 1) (at 226.695 95.885 0)
       (effects (font (size 1.27 1.27)) (justify left))
     )
@@
     (in_bom yes) (on_board yes) (fields_autoplaced)
     (property "Reference" "R38" (id 0) (at 36.83 98.7892 90))
-    (property "Value" "37.4" (id 1) (at 36.83 101.3261 90))
+    (property "Value" "37.4R" (id 1) (at 36.83 101.3261 90))
     (property "Footprint" "Resistor_SMD:R_0603_1608Metric" (id 2) (at 36.83 101.727 90)
       (effects (font (size 1.27 1.27)) hide)
@@
       (effects (font (size 1.27 1.27)) (justify left))
     )
-    (property "Value" "150" (id 1) (at 185.42 116.84 0)
+    (property "Value" "150R" (id 1) (at 185.42 116.84 0)
       (effects (font (size 1.27 1.27)) (justify left))
     )
@@
       (effects (font (size 1.27 1.27)) (justify left))
     )
-    (property "Value" "150" (id 1) (at 43.688 110.9222 0)
+    (property "Value" "150R" (id 1) (at 43.688 110.9222 0)
       (effects (font (size 1.27 1.27)) (justify left))
     )
@@
       (effects (font (size 1.27 1.27)) (justify left))
     )
-    (property "Value" "150" (id 1) (at 33.528 110.9222 0)
+    (property "Value" "150R" (id 1) (at 33.528 110.9222 0)
       (effects (font (size 1.27 1.27)) (justify left))
     )
@@
   )
   (symbol (lib_id "Device:L") (at 268.605 121.92 0) (unit 1)
-    (in_bom yes) (on_board yes) (fields_autoplaced)
-    (property "Reference" "L12" (id 0) (at 269.875 121.0853 0)
-      (effects (font (size 1.27 1.27)) (justify left))
-    )
-    (property "Value" "1u" (id 1) (at 269.875 123.6222 0)
+    (in_bom yes) (on_board yes)
+    (property "Reference" "L12" (id 0) (at 269.875 120.015 0)
+      (effects (font (size 1.27 1.27)) (justify left))
+    )
+    (property "Value" "1u" (id 1) (at 265.43 123.825 0)
       (effects (font (size 1.27 1.27)) (justify left))
     )
@@
       (effects (font (size 1.27 1.27)) (justify left))
     )
-    (property "Value" "150" (id 1) (at 220.98 95.885 0)
+    (property "Value" "150R" (id 1) (at 220.98 95.885 0)
       (effects (font (size 1.27 1.27)) (justify left))
     )
@@
       (effects (font (size 1.27 1.27)) (justify left))
     )
-    (property "Value" "150" (id 1) (at 191.135 116.84 0)
-      (effects (font (size 1.27 1.27)) (justify left))
-    )
+    (property "Value" "150R" (id 1) (at 191.135 116.84 0)
+      (effects (font (size 1.27 1.27)) (justify left))
+    )

Commit message: Merge branch 'main' of https://github.com/M0LTE/pi-transceiver
Addition of PA Board version 2 Kicad files
Parts:
- C31: footprint Capacitor_SMD:CP_Elec_8x6.7 -> Capacitor_Tantalum_SMD:CP_EIA-7360-38_Kemet-E
Other:
- note added: "6dB Attenuator"
