File: electronics/PA_Board/Pi_TX_35W_PA.kicad_sch (KiCad schematic)
At the start: 5 parts

Commit message: PCB updates and gerbers
Parts:
- removed H1, H2, H3, H4: MountingHole, MountingHole:MountingHole_4.3mm_M4, symbol Mechanical:MountingHole
- added H1, H2, H3, H4: MountingHole_Pad, MountingHole:MountingHole_4.3mm_M4_DIN965_Pad, symbol Mechanical:MountingHole_Pad
- added LOGO1: Logo_Open_Hardware_Small, Symbol:OSHW-Logo2_9.8x8mm_SilkScreen, symbol Graphic:Logo_Open_Hardware_Small
Connections:
- new net GND: H1.1, H2.1, H3.1, H4.1
Other:
- sheet PA_Power ports: added none; removed VDD_GAIN
- sheet PA_RF ports: added none; removed VDD_GAIN
