File: electronics/receiver/PIN_SW.kicad_sch (KiCad schematic)
At the start: 35 parts, among them J401 Conn_Coaxial, J402 Conn_Coaxial, J403 Conn_Coaxial, J404 Conn_01x06_Male, J405 Conn_01x01_Male, J406 Conn_Coaxial, U401 AS179-92LF, U402 AS179-92LF, U403 AMS1117-5.0, U404 AS179-92LF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

Commit message: Branch for changes to RX LNA board from M0SKP
Upgrade files to Kicad 7
Added Fields for comment and LCSC part numbers to symbol table
Populated some LCSC part numbers to allow testing at JLCPCB
Parts:
- C401, C402, C403, C404, C410, C412: Comment (none) -> Ceramic Capacitor 1nf 50V 5% 0805; LCSC Part (none) -> C62774
- C405, C406, C407, C408: Comment (none) -> Ceramic Capacitor 100pf 50V 5% 0805; LCSC Part (none) -> C62768
- C409, C411: Comment (none) -> Ceramic Capacitor 100nf 50V 5% 0805; LCSC Part (none) -> C111492
- U401, U402, U404: Comment (none) -> SPDT RF Switch SOT363; LCSC Part (none) -> C83422
- U403: Comment (none) -> Voltage Regulator Fixed 5V SOT223-3; LCSC Part (none) -> C917153
- U405: Comment (none) -> Voltage Regulator Fixed 3.3V SOT223-3; LCSC Part (none) -> C5199435
- U406: Comment (none) -> I2C IO Expander SOP16; LCSC Part (none) -> C86832
