File: electronics/receiver/RXLNA.kicad_pcb (KiCad board)
At the start: 4 copper layers, 100 x 100 mm, 86 parts, among them J401 Conn_Coaxial, J402 Conn_Coaxial, J403 Conn_Coaxial, J404 Conn_01x06_Male, J405 Conn_01x01_Male, J406 Conn_Coaxial, J407 Conn_Coaxial, U401 AS179-92LF, U402 AS179-92LF, U403 AMS1117-5.0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

Commit message: Branch for changes to RX LNA board from M0SKP
Upgrade files to Kicad 7
Added Fields for comment and LCSC part numbers to symbol table
Populated some LCSC part numbers to allow testing at JLCPCB
Parts:
- C401, C402, C403, C404, C410, C412, C413, C414, C415, C416, C419, C421, C422, C423, C424: value C -> 1n0
- C405, C406, C407, C408: value C -> 100p
- C409, C411, C420: value C -> 100n
- C425: value C -> 15p
- C426, C430, C445: value C -> 6p8
- C427: value C -> 8p2
- C428: value C -> 18p
- C429, C434, C439, C444: value C_Trim -> 5-22pF
- C431: value C -> 0p7
- C432, C437, C442: value C -> 12p0
- C433, C438: value C -> 22p0
- C435: value C -> 0p9
- C436, C441: value C -> 0p5
- C440: value C -> 1p8
- C443: value C -> 15p0
- C446: value C -> 3p9
- L403, L404, L405, L406: value L -> 54n6
