File: electronics/receiver/BPF.kicad_sch (KiCad schematic)
At the start: 26 parts

Commit message: Update values
Parts:
- C425: value 15p -> 11p
- C426: value 6p8 -> 9p1
- C430: value 6p8 -> 4p7
- C431: value 0p7 -> 0p5
- C435: value 0p9 -> 1p
- C440: value 1p8 -> 2p2
- C445: value 6p8 -> 10p
- C446: value 3p9 -> 3p6
- L403, L404, L405, L406: value 54n6 -> 54n58
Changed lines of the file:
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@@
     (stroke (width 0) (type default) (color 0 0 0 0))
+  )
+  (label "15.759pF" (at 151.13 113.03 0)
+    (effects (font (size 1.27 1.27)) (justify left bottom))
+  )
+  (label "144 - 147 MHz bandwidth, Attenuation 2dB" (at 123.19 67.31 0)
+    (effects (font (size 1.27 1.27)) (justify left bottom))
+  )
+  (label "Nominal trimmer values" (at 50.8 113.03 0)
+    (effects (font (size 1.27 1.27)) (justify left bottom))
+  )
+  (label "15.066pF" (at 120.65 113.03 0)
+    (effects (font (size 1.27 1.27)) (justify left bottom))
+  )
+  (label "14.712pF" (at 83.82 113.03 0)
+    (effects (font (size 1.27 1.27)) (justify left bottom))
+  )
+  (label "12.668pF" (at 196.85 113.03 0)
+    (effects (font (size 1.27 1.27)) (justify left bottom))
   )
   (global_label "BPF_Out" (shape input) (at 227.33 86.36 0) (fields_autoplaced)
@@
     (in_bom yes) (on_board yes) (fields_autoplaced)
     (property "Reference" "C440" (id 0) (at 180.34 78.74 90))
-    (property "Value" "1p8" (id 1) (at 180.34 81.28 90))
+    (property "Value" "2p2" (id 1) (at 180.34 81.28 90))
     (property "Footprint" "Capacitor_SMD:C_0603_1608Metric_Pad1.08x0.95mm_HandSolder" (id 2) (at 176.53 87.3252 0)
       (effects (font (size 1.27 1.27)) hide)
@@
     (in_bom yes) (on_board yes) (fields_autoplaced)
     (property "Reference" "C430" (id 0) (at 102.87 78.74 90))
-    (property "Value" "6p8" (id 1) (at 102.87 81.28 90))
+    (property "Value" "4p7" (id 1) (at 102.87 81.28 90))
     (property "Footprint" "Capacitor_SMD:C_0603_1608Metric_Pad1.08x0.95mm_HandSolder" (id 2) (at 99.06 87.3252 0)
       (effects (font (size 1.27 1.27)) hide)
@@
       (effects (font (size 1.27 1.27)) (justify left))
     )
-    (property "Value" "54n6" (id 1) (at 138.43 97.7899 0)
+    (property "Value" "54n58" (id 1) (at 138.43 97.7899 0)
       (effects (font (size 1.27 1.27)) (justify left))
     )
@@
       (effects (font (size 1.27 1.27)) (justify left))
     )
-    (property "Value" "54n6" (id 1) (at 176.53 99.0599 0)
+    (property "Value" "54n58" (id 1) (at 176.53 99.0599 0)
       (effects (font (size 1.27 1.27)) (justify left))
     )
@@
     (in_bom yes) (on_board yes) (fields_autoplaced)
     (property "Reference" "C446" (id 0) (at 223.52 78.74 90))
-    (property "Value" "3p9" (id 1) (at 223.52 81.28 90))
+    (property "Value" "3p6" (id 1) (at 223.52 81.28 90))
     (property "Footprint" "Capacitor_SMD:C_0603_1608Metric_Pad1.08x0.95mm_HandSolder" (id 2) (at 219.71 87.3252 0)
       (effects (font (size 1.27 1.27)) hide)
@@
     (in_bom yes) (on_board yes) (fields_autoplaced)
     (property "Reference" "C425" (id 0) (at 66.04 78.74 90))
-    (property "Value" "15p" (id 1) (at 66.04 81.28 90))
+    (property "Value" "11p" (id 1) (at 66.04 81.28 90))
     (property "Footprint" "Capacitor_SMD:C_0603_1608Metric_Pad1.08x0.95mm_HandSolder" (id 2) (at 62.23 87.3252 0)
       (effects (font (size 1.27 1.27)) hide)
@@
       (effects (font (size 1.27 1.27)) (justify left))
     )
-    (property "Value" "54n6" (id 1) (at 214.63 99.0599 0)
+    (property "Value" "54n58" (id 1) (at 214.63 99.0599 0)
       (effects (font (size 1.27 1.27)) (justify left))
     )
@@
     (in_bom yes) (on_board yes) (fields_autoplaced)
     (property "Reference" "C435" (id 0) (at 140.97 78.74 90))
-    (property "Value" "0p9" (id 1) (at 140.97 81.28 90))
+    (property "Value" "1p" (id 1) (at 140.97 81.28 90))
     (property "Footprint" "Capacitor_SMD:C_0603_1608Metric_Pad1.08x0.95mm_HandSolder" (id 2) (at 137.16 87.3252 0)
       (effects (font (size 1.27 1.27)) hide)
@@
       (effects (font (size 1.27 1.27)) (justify left))
     )
-    (property "Value" "54n6" (id 1) (at 100.33 99.0599 0)
+    (property "Value" "54n58" (id 1) (at 100.33 99.0599 0)
       (effects (font (size 1.27 1.27)) (justify left))
     )
@@
     (in_bom yes) (on_board yes) (fields_autoplaced)
     (property "Reference" "C431" (id 0) (at 109.22 78.74 90))
-    (property "Value" "0p7" (id 1) (at 109.22 81.28 90))
+    (property "Value" "0p5" (id 1) (at 109.22 81.28 90))
     (property "Footprint" "Capacitor_SMD:C_0603_1608Metric_Pad1.08x0.95mm_HandSolder" (id 2) (at 105.41 87.3252 0)
       (effects (font (size 1.27 1.27)) hide)
@@
     (in_bom yes) (on_board yes) (fields_autoplaced)
     (property "Reference" "C426" (id 0) (at 72.39 78.74 90))
-    (property "Value" "6p8" (id 1) (at 72.39 81.28 90))
+    (property "Value" "9p1" (id 1) (at 72.39 81.28 90))
     (property "Footprint" "Capacitor_SMD:C_0603_1608Metric_Pad1.08x0.95mm_HandSolder" (id 2) (at 68.58 87.3252 0)
       (effects (font (size 1.27 1.27)) hide)
@@
     (in_bom yes) (on_board yes) (fields_autoplaced)
     (property "Reference" "C445" (id 0) (at 217.17 78.74 90))
-    (property "Value" "6p8" (id 1) (at 217.17 81.28 90))
+    (property "Value" "10p" (id 1) (at 217.17 81.28 90))
     (property "Footprint" "Capacitor_SMD:C_0603_1608Metric_Pad1.08x0.95mm_HandSolder" (id 2) (at 213.36 87.3252 0)
       (effects (font (size 1.27 1.27)) hide)
