File: electronics/receiver/BPF.kicad_sch (KiCad schematic)
At the start: 26 parts

Commit message: Repair
Fix Github commit problem
Parts:
- C428: renamed from C425; value 11p -> 68p
- C429: renamed from C426; value 9p1 -> 8p2
- C430: renamed from C427; value 8p2 -> 1p2
- C431: renamed from C428; value 18p -> 10p
- C432: renamed from C429; value 5-22pF -> 2-10pF
- C433: renamed from C430; value 4p7 -> 1n
- C434: renamed from C431; value 0p5 -> 1p3
- C435: renamed from C432; value 12p0 -> 8p2
- C436: renamed from C433; value 22p0 -> 10p0
- C437: renamed from C434; value 5-22pF -> 2-10pF
- C438: renamed from C435; value 1p -> 1n
- C439: renamed from C436; value 0p5 -> 0p7
- C440: renamed from C437; value 12p0 -> 8p2
- C441: renamed from C438; value 22p0 -> 10p0
- C442: renamed from C439; value 5-22pF -> 2-10pF
- C443: renamed from C440; value 2p2 -> 1n
- C444: renamed from C441; value 0p5 -> 0p8
- C445: renamed from C442; value 12p0 -> 6p2
- C446: renamed from C443; value 15p0 -> 10p0
- C447: renamed from C444; value 5-22pF -> 2-10pF
- C448: renamed from C445; value 10p -> 4p3
- C449: renamed from C446; value 3p6 -> 1n
