File: electronics/PA_Board_V2/Pi_TX_35W_PA_V2.kicad_pcb (KiCad board)
At the start: 4 copper layers, 100 x 100 mm, 166 parts, among them J1 USB_B_Micro, J10 Conn_01x04, J2 Conn_01x05, J3 Conn_01x05, J4 Conn_01x04, J5 Conn_01x02, J6 Conn_Coaxial, J7 Conn_Coaxial, J8 Conn_Coaxial, J9 Conn_Coaxial, K1 G6E, Q1 AOD4185, Q2 BC848W, Q3 2N7002, SW1 SW_Push, U1 ATSAMD21E18A-A, U10 RA35H1516M, U11 Directional_Coupler, U12 74LV1T34, U2 LM75B, U3 LM2904, U4 LMR51420, U5 MCP4725, U6 AP2204K-ADJ, U7 TLV70233, U8 INA219AxD, U9 ADL5611

Commit message: Add RF Screen and some PCB and BOM changes
Parts:
- removed Q3: 2N7002, Package_TO_SOT_SMD:SOT-23
- removed R49: 2k, Resistor_SMD:R_0603_1608Metric
- removed R50: 10k, Resistor_SMD:R_0603_1608Metric
- added F1: 1A, Fuse:Fuse_1206_3216Metric, F.Cu at (144.2, 84.6)
- added F2: 150mA, Fuse:Fuse_0805_2012Metric, F.Cu at (112.8, 133.8)
- added F3: 150mA, Fuse:Fuse_0805_2012Metric, F.Cu at (112.8, 136.1)
- added F4: 150mA, Fuse:Fuse_0805_2012Metric, F.Cu at (112.8, 138.5)
- added U13: 74LV1T34, Package_TO_SOT_SMD:SOT-353_SC-70-5, F.Cu at (113.4, 100.5)
- H1, H2, H3, H4: footprint MountingHole:MountingHole_4.3mm_M4_DIN965_Pad -> MountingHole:MountingHole_3.2mm_M3_DIN965_Pad
- J4: value Conn_01x04 -> Conn_01x06; footprint Pi_Tx_V2:JST_PH_S4B-PH-SM4-TB_1x04-1MP_P2.00mm_Horizontal -> Pi_Tx_V2:JST_PH_S6B-PH-SM4-TB_1x06-1MP_P2.00mm_Horizontal
- moved J4 0.91 mm to (105.0, 130.2)
- moved J3 0.89 mm to (105.1, 112.3)
Connections:
- D5 pad 4: +3.3V -> Net-(J4-Pin_3)
- J4 pad 3: +3.3V -> Net-(J4-Pin_3)
- Q1 pad 3: +12V -> /PA_Power/VBAT
- R36 pad 2: +12V -> /PA_Power/VBAT
- R51 pad 2: Net-(Q3-D) -> /PA_Protection/Fan_RPM
- R52 pad 1: +12V -> /PA_Power/VBAT
Routing:
- net /PA_Power/VBAT: track 0.00 -> 39.6 mm, vias 0 -> 12
- net +5V: track 79.7 -> 115.3 mm, vias 2 -> 4
- net VDC: track 96.9 -> 114.7 mm
- net GND: track 283.5 -> 274.5 mm, vias 351 -> 350
- net Net-(Q3-D): track 8.30 -> 0.00 mm
- net Net-(J4-Pin_3): track 0.00 -> 7.34 mm
- net +3.3V: track 70.9 -> 64.6 mm
- net Net-(J4-Pin_6): track 0.00 -> 5.38 mm
- net +12V: track 170.5 -> 175.8 mm, vias 19 -> 8
- net Net-(J4-Pin_5): track 0.00 -> 5.21 mm
- net /PA_Protection/Fan_RPM: track 38.7 -> 42.4 mm, vias 1 -> 2
- net Net-(J10-Pin_4): track 3.68 -> 6.67 mm
- net Net-(J2-Pin_5): track 49.3 -> 50.8 mm
- net /PA_Protection/Fan PWM: track 38.8 -> 40.3 mm
- added copper zone on B.Cu, net /PA_Power/VBAT
- added copper zone on F.Cu, net /PA_Power/VBAT
- added copper zone on In1.Cu, net /PA_Power/VBAT
- added copper zone on In2.Cu, net /PA_Power/VBAT
- removed copper zone on B.Cu, net +12V
- removed copper zone on F.Cu, net +12V
- removed copper zone on In1.Cu, net +12V
- removed copper zone on In2.Cu, net +12V
Other:
- board text added: "I2C/Power"
- board text removed: "I2C"

Commit message: Latest version
Parts:
- added C1: 100p, Capacitor_SMD:C_0603_1608Metric, F.Cu at (113.3, 88.1)
- added C21: 1u, Capacitor_SMD:C_0603_1608Metric, F.Cu at (112.9, 90.3)
- added C4: 100n, Capacitor_SMD:C_0603_1608Metric, F.Cu at (113.2, 86.4)
- added C61: 9p1, Capacitor_SMD:C_1206_3216Metric, F.Cu at (170.5, 87.5)
- added C62: 3p, Capacitor_SMD:C_1206_3216Metric, F.Cu at (170.2, 99.2)
- added C63: 6p8, Capacitor_SMD:C_1206_3216Metric, F.Cu at (163.5, 101.0)
- added C9: 330p, Capacitor_SMD:C_0603_1608Metric, F.Cu at (116.3, 83.4)
- added L1: 1u, Inductor_SMD:L_0805_2012Metric, F.Cu at (116.1, 87.1)
- added R10: 10k, Resistor_SMD:R_0603_1608Metric, F.Cu at (112.9, 92.3)
- added R48: 300R, Resistor_SMD:R_0603_1608Metric, F.Cu at (118.0, 83.6)
- added R49: 18R, Resistor_SMD:R_0603_1608Metric, F.Cu at (118.0, 80.4)
- added R50: 300R, Resistor_SMD:R_0603_1608Metric, F.Cu at (118.0, 77.3)
- added U1: PSA4-5043+, Pi_Tx_V2:MM1362 PSA4-5043+, F.Cu at (113.7, 83.3)
- added U8: TPS22810DBV, Package_TO_SOT_SMD:SOT-23-6, F.Cu at (116.5, 91.2)
- C3: renamed from C29; value 10n -> 330p
- R2: renamed from R38; value 37.4R -> 18R
- R3: renamed from R39; value 150R -> 300R
- R4: renamed from R37; value 150R -> 300R
- U14: renamed from U11; footprint Pi_Tx_V2:Wiggly Coupler -> Pi_Tx_V2:Linear_Coupler
- U3: renamed from U9; value ADL5611 -> PSA4-5043+; footprint Package_TO_SOT_SMD:SOT-89-3 -> Pi_Tx_V2:MM1362 PSA4-5043+
- moved C20 12.7 mm to (175.1, 99.2)
- moved R40 9.70 mm to (157.6, 110.4), turned to -151 degrees
- moved C47 9.08 mm to (161.6, 125.0), turned to 180 degrees
- moved R38 8.94 mm to (156.9, 109.1), turned to -151 degrees
- moved LOGO1 7.55 mm to (153.6, 119.2)
- moved C35 6.89 mm to (167.3, 108.2), turned to 0 degrees
- moved C36 6.63 mm to (167.4, 104.3), turned to 180 degrees
- moved L10 5.82 mm to (161.5, 126.8)
- moved D12 5.64 mm to (165.3, 124.3), turned to 29 degrees
- moved R22 5.58 mm to (171.4, 121.2), turned to -151 degrees
- moved L8 5.45 mm to (167.3, 106.2)
- moved R3 5.45 mm to (107.0, 87.6), turned to -90 degrees
- moved C32 5.40 mm to (149.9, 100.5), turned to 180 degrees
- moved D3 4.98 mm to (163.4, 106.8), turned to -151 degrees
- moved D11 4.69 mm to (166.0, 125.5), turned to -151 degrees
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- renumbered C28 to C10, C37 to C11, C43 to C12, C31 to C13, C33 to C14, C42 to C15, C36 to C16, C56 to C17, C27 to C18, C38 to C19, C9 to C2, C41 to C20, C20 to C22, C13 to C23, C8 to C24, C16 to C25, C19 to C26, C15 to C27, C22 to C28, C18 to C29, C26 to C30, C17 to C31, C45 to C32, C39 to C33, C40 to C34, C44 to C35, C47 to C36, C1 to C37, C23 to C38, C7 to C39, C4 to C40, C21 to C41, C14 to C42, C11 to C43, C6 to C44, C3 to C45, C25 to C46, C51 to C47, C10 to C48, C24 to C49, C35 to C5, C12 to C50, C48 to C51, C55 to C52, C2 to C53, C5 to C54, C52 to C55, C54 to C56, C46 to C57, C49 to C58, C50 to C59, C32 to C6, C53 to C60, C30 to C7, C34 to C8, D4 to D1, D6 to D10, D15 to D11, D14 to D12, D3 to D13, D19 to D14, D18 to D15, D17 to D16, D16 to D17, D13 to D2, D12 to D3, D11 to D4, D7 to D6, D9 to D7, D1 to D8, D10 to D9, H3 to H1, H1 to H3, J6 to J1, J2 to J10, J10 to J2, J5 to J4, J7 to J5, J4 to J6, J9 to J7, J1 to J9, L9 to L10, L10 to L12, L12 to L13, L4 to L2, L5 to L3, L3 to L4, L2 to L5, L7 to L6, L6 to L7, L1 to L9, R9 to R1, R51 to R11, R35 to R12, R33 to R13, R34 to R14, R32 to R15, R4 to R16, R31 to R17, R8 to R18, R15 to R19, R30 to R20, R12 to R21, R44 to R22, R45 to R23, R10 to R24, R11 to R25, R24 to R26, R13 to R27, R20 to R28, R16 to R29, R23 to R30, R18 to R31, R17 to R32, R14 to R33, R19 to R34, R21 to R35, R25 to R36, R22 to R37, R41 to R38, R42 to R39, R43 to R41, R3 to R42, R1 to R43, R2 to R44, R46 to R45, R48 to R46, R7 to R5, R53 to R7, R52 to R8, R36 to R9, U8 to U10, U7 to U11, U3 to U12, U1 to U13, U12 to U15, U10 to U4, U13 to U5, U4 to U6, U5 to U7, U6 to U9
Connections:
- C10 pad 2: +5V -> Net-(U8-VOUT)
- C12 pad 1: Net-(C41-Pad2) -> Net-(C12-Pad1)
- C15 pad 1: Net-(C41-Pad2) -> Net-(C12-Pad1)
- C19 pad 1: Net-(U10-RF_Out) -> Net-(C19-Pad1)
- C20 pad 2: Net-(C41-Pad2) -> Net-(C20-Pad2)
- C3 pad 1: Net-(C29-Pad1) -> Net-(C3-Pad1)
- C5 pad 2: Net-(C35-Pad2) -> Net-(C5-Pad2)
- C7 pad 2: +5V -> Net-(U8-VOUT)
- L2 pad 1: +5V -> Net-(U8-VOUT)
- L2 pad 2: Net-(C35-Pad2) -> Net-(C5-Pad2)
- L3 pad 1: Net-(U10-RF_Out) -> Net-(U4-RF_Out)
- L6 pad 1: Net-(C41-Pad2) -> Net-(C12-Pad1)
- L7 pad 2: Net-(C41-Pad2) -> Net-(C12-Pad1)
- U13 pad 8: unconnected-(U1-PA07-Pad8) -> /PA_Protection/DRIVER_EN
- U3 pad 1: Net-(C29-Pad1) -> Net-(C5-Pad2)
- U3 pad 3: Net-(C35-Pad2) -> Net-(R49-Pad1)
- U4 pad 4: Net-(U10-RF_Out) -> Net-(U4-RF_Out)
Routing:
- net /PA_Protection/DRIVER_EN: track 0.00 -> 47.6 mm, vias 0 -> 2
- net Net-(C41-Pad2): track 23.0 -> 0.00 mm
- net GND: track 274.5 -> 252.1 mm, vias 350 -> 416
- net Net-(U4-RF_Out): track 0.00 -> 22.0 mm
- net Net-(C12-Pad1): track 0.00 -> 21.8 mm
- net Net-(U14-RF): track 9.73 -> 29.8 mm
- net Net-(U10-RF_Out): track 19.2 -> 0.00 mm
- net Net-(U8-VOUT): track 0.00 -> 17.0 mm
- net +5V: track 115.3 -> 109.7 mm
- net Net-(C5-Pad2): track 0.00 -> 4.83 mm
- net Net-(C29-Pad1): track 4.64 -> 0.00 mm
- net Net-(C35-Pad2): track 4.31 -> 0.00 mm
- net /PA_Protection/VRev: track 17.9 -> 22.0 mm
- net Net-(C9-Pad2): track 0.00 -> 3.69 mm
- net /PA_Protection/Fan PWM: track 40.3 -> 43.8 mm
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Other:
- board text added: "TX Monitor"
- board text added: "V2.0 Dec. 2023"
- board text added: "www.radarc.org"
- board text removed: "Tx Monitor"
- board text removed: "V2.0"
- board text removed: "www.radarc.org Nov. 2023"
