File: electronics/PA_Board_V2/Pi_TX_35W_PA_V2.kicad_sch (KiCad schematic)
At the start: 6 parts

Commit message: Add RF Screen and some PCB and BOM changes
Parts:
- H1, H2, H3, H4: footprint MountingHole:MountingHole_4.3mm_M4_DIN965_Pad -> MountingHole:MountingHole_3.2mm_M3_DIN965_Pad
Changed lines of the file:
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@@
       (effects (font (size 1.27 1.27)) (justify left))
     )
-    (property "Footprint" "MountingHole:MountingHole_4.3mm_M4_DIN965_Pad" (at 72.39 176.53 0)
+    (property "Footprint" "MountingHole:MountingHole_3.2mm_M3_DIN965_Pad" (at 72.39 176.53 0)
       (effects (font (size 1.27 1.27)) hide)
     )
@@
       (effects (font (size 1.27 1.27)) (justify left))
     )
-    (property "Footprint" "MountingHole:MountingHole_4.3mm_M4_DIN965_Pad" (at 72.39 165.1 0)
+    (property "Footprint" "MountingHole:MountingHole_3.2mm_M3_DIN965_Pad" (at 72.39 165.1 0)
       (effects (font (size 1.27 1.27)) hide)
     )
@@
       (effects (font (size 1.27 1.27)) (justify left))
     )
-    (property "Footprint" "MountingHole:MountingHole_4.3mm_M4_DIN965_Pad" (at 72.39 170.815 0)
+    (property "Footprint" "MountingHole:MountingHole_3.2mm_M3_DIN965_Pad" (at 72.39 170.815 0)
       (effects (font (size 1.27 1.27)) hide)
     )
@@
       (effects (font (size 1.27 1.27)) (justify left))
     )
-    (property "Footprint" "MountingHole:MountingHole_4.3mm_M4_DIN965_Pad" (at 72.39 182.245 0)
+    (property "Footprint" "MountingHole:MountingHole_3.2mm_M3_DIN965_Pad" (at 72.39 182.245 0)
       (effects (font (size 1.27 1.27)) hide)
     )

Commit message: Latest version
Parts:
- renumbered H3 to H1, H1 to H3
Other:
- sheet PA_Protection ports: added DRIVER_EN; removed none
- sheet PA_RF ports: added DRIVER_EN; removed none
Changed lines of the file:
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@@
+    (stroke (width 0) (type default))
+  )
+  (wire (pts (xy 175.26 82.55) (xy 175.26 114.3))
     (stroke (width 0) (type default))
   )
@@
   (symbol (lib_id "Mechanical:MountingHole_Pad") (at 72.39 176.53 270) (unit 1)
     (in_bom no) (on_board yes) (dnp no) (fields_autoplaced)
-    (property "Reference" "H3" (at 76.2 175.6953 90)
+    (property "Reference" "H1" (at 76.2 175.6953 90)
       (effects (font (size 1.27 1.27)) (justify left))
     )
@@
       (project "Pi_TX_35W_PA_V2"
         (path "/296f23ba-4d28-4f71-91fa-c9ce5a8d0c63"
+          (reference "H1") (unit 1)
+        )
+      )
+    )
+  )
+  (symbol (lib_id "Mechanical:MountingHole_Pad") (at 72.39 165.1 270) (unit 1)
+    (in_bom no) (on_board yes) (dnp no) (fields_autoplaced)
+    (property "Reference" "H3" (at 76.2 164.2653 90)
+      (effects (font (size 1.27 1.27)) (justify left))
+    )
+    (property "Value" "MountingHole_Pad" (at 76.2 166.8022 90)
+      (effects (font (size 1.27 1.27)) (justify left))
+    )
+    (property "Footprint" "MountingHole:MountingHole_3.2mm_M3_DIN965_Pad" (at 72.39 165.1 0)
+      (effects (font (size 1.27 1.27)) hide)
+    )
+    (property "Datasheet" "~" (at 72.39 165.1 0)
+      (effects (font (size 1.27 1.27)) hide)
+    )
+    (property "Comment" "not fitted" (at 72.39 165.1 0)
+      (effects (font (size 1.27 1.27)) hide)
+    )
+    (property "LCSC Part" "" (at 72.39 165.1 0)
+      (effects (font (size 1.27 1.27)) hide)
+    )
+    (pin "1")
+    (instances
+      (project "Pi_TX_35W_PA_V2"
+        (path "/296f23ba-4d28-4f71-91fa-c9ce5a8d0c63"
           (reference "H3") (unit 1)
-        )
-      )
-    )
-  )
-  (symbol (lib_id "Mechanical:MountingHole_Pad") (at 72.39 165.1 270) (unit 1)
-    (in_bom no) (on_board yes) (dnp no) (fields_autoplaced)
-    (property "Reference" "H1" (at 76.2 164.2653 90)
-      (effects (font (size 1.27 1.27)) (justify left))
-    )
-    (property "Value" "MountingHole_Pad" (at 76.2 166.8022 90)
-      (effects (font (size 1.27 1.27)) (justify left))
-    )
-    (property "Footprint" "MountingHole:MountingHole_3.2mm_M3_DIN965_Pad" (at 72.39 165.1 0)
-      (effects (font (size 1.27 1.27)) hide)
-    )
-    (property "Datasheet" "~" (at 72.39 165.1 0)
-      (effects (font (size 1.27 1.27)) hide)
-    )
-    (property "Comment" "not fitted" (at 72.39 165.1 0)
-      (effects (font (size 1.27 1.27)) hide)
-    )
-    (property "LCSC Part" "" (at 72.39 165.1 0)
-      (effects (font (size 1.27 1.27)) hide)
-    )
-    (pin "1")
-    (instances
-      (project "Pi_TX_35W_PA_V2"
-        (path "/296f23ba-4d28-4f71-91fa-c9ce5a8d0c63"
-          (reference "H1") (unit 1)
         )
       )
@@
       (effects (font (size 1.27 1.27)) (justify left))
     )
+    (pin "DRIVER_EN" output (at 175.26 82.55 270)
+      (effects (font (size 1.27 1.27)) (justify left))
+    )
     (instances
       (project "Pi_TX_35W_PA_V2"
@@
       (effects (font (size 1.27 1.27)) (justify left))
     )
-    (instances
+    (pin "DRIVER_EN" input (at 175.26 114.3 90)
+      (effects (font (size 1.27 1.27)) (justify right))
+    )
+    (instances
