File: electronics/PA_Board_V2/PA_Power_V2.kicad_sch (KiCad schematic)
At the start: 35 parts, among them J5 Conn_01x02, Q1 AOD4185, U4 LMR51420, U5 MCP4725, U6 AP2204K-ADJ, U7 TLV70233, U8 INA219AxD

Commit message: Update PA board V2 Kicad files
New schematic, PCB, and footprints
Parts:
- added F1: 1A, Fuse:Fuse_1206_3216Metric, symbol Device:Polyfuse
- J4: renamed from J5; Comment (none) -> not fitted; now left out of the parts list
- R7: renamed from R53; value 10k -> 10R; LCSC Part C25804 -> C22859
- R8: renamed from R52; value 10k -> 10R; LCSC Part C25804 -> C22859
- renumbered C56 to C17, C20 to C22, C13 to C23, C16 to C25, C19 to C26, C15 to C27, C22 to C28, C18 to C29, C26 to C30, C17 to C31, C23 to C38, C21 to C41, C14 to C42, C25 to C46, C24 to C49, D11 to D4, D9 to D7, D10 to D9, L2 to L5, R35 to R12, R33 to R13, R34 to R14, R32 to R15, R31 to R17, R30 to R20, R36 to R9, U8 to U10, U7 to U11, U4 to U6, U5 to U7, U6 to U9
Connections:
- net +12V: now also F1.2; no longer Q1.3 (S), R8.1, R9.2
- net GND: now also U7.6 (A0)
- new net VBAT: F1.1, Q1.3 (S), R8.1, R9.2
- no-connect marks 1 -> 0
Other:
- note added: "I2C Address 0x60"
- note removed: "I2C Address 0x61"
