File: electronics/PA_Board_V2/PA_RF_V2.kicad_sch (KiCad schematic)
At the start: 65 parts, among them J6 Conn_Coaxial, J7 Conn_Coaxial, J8 Conn_Coaxial, J9 Conn_Coaxial, K1 G6E, Q2 BC848W, U10 RA35H1516M, U11 Directional_Coupler, U9 ADL5611

Commit message: Update PA board V2 Kicad files
New schematic, PCB, and footprints
Parts:
- added C1: 100p, Capacitor_SMD:C_0603_1608Metric, symbol Device:C
- added C21: 1u, Capacitor_SMD:C_0603_1608Metric, symbol Device:C
- added C4: 100n, Capacitor_SMD:C_0603_1608Metric, symbol Device:C
- added C61: 9p1, Capacitor_SMD:C_1206_3216Metric, symbol Device:C
- added C62: 3p, Capacitor_SMD:C_1206_3216Metric, symbol Device:C
- added C63: 6p8, Capacitor_SMD:C_1206_3216Metric, symbol Device:C
- added C64, C9: 330p, Capacitor_SMD:C_0603_1608Metric, symbol Device:C
- added L1: 1u, Inductor_SMD:L_0805_2012Metric, symbol Device:L
- added R10: 10k, Resistor_SMD:R_0603_1608Metric, symbol Device:R
- added R48, R50: 300R, Resistor_SMD:R_0603_1608Metric, symbol Device:R
- added R49: 18R, Resistor_SMD:R_0603_1608Metric, symbol Device:R
- added U1: PSA4-5043+, Pi_Tx_V2:MM1362 PSA4-5043+, symbol Pi_PA:PSA4-5043+
- added U8: TPS22810DBV, Package_TO_SOT_SMD:SOT-23-6, symbol Pi_PA:TPS22810DBV
- C3: renamed from C29; value 10n -> 330p; Comment 10n 0603 50V 2% -> 330p 0603 50V 2%; LCSC Part C2215227 -> C458903
- J1: renamed from J6; LCSC Part C1509221 -> C496550
- J5: renamed from J7; LCSC Part C1509221 -> C496550
- J7: renamed from J9; LCSC Part C1509221 -> C496550
- J8: LCSC Part C1509221 -> C496550
- L11: LCSC Part C1042 -> C703134
- L12: renamed from L10; LCSC Part C1042 -> C703134
- L13: renamed from L12; LCSC Part C1042 -> C703134
- L2: renamed from L4; LCSC Part C1042 -> C703134
- R2: renamed from R38; value 37.4R -> 18R; LCSC Part C2933689 -> C245924
- R3: renamed from R39; value 150R -> 300R; LCSC Part C22808 -> C2930092
- R4: renamed from R37; value 150R -> 300R; LCSC Part C22808 -> C2930092
- U14: renamed from U11; footprint Pi_Tx_V2:Wiggly Coupler -> Pi_Tx_V2:Linear_Coupler
- U3: renamed from U9; value ADL5611 -> PSA4-5043+; footprint Package_TO_SOT_SMD:SOT-89-3 -> Pi_Tx_V2:MM1362 PSA4-5043+; symbol RF_Amplifier:SPF5189Z -> Pi_PA:PSA4-5043+; LCSC Part C208262 -> C5240848
- renumbered C28 to C10, C37 to C11, C43 to C12, C31 to C13, C33 to C14, C42 to C15, C36 to C16, C27 to C18, C38 to C19, C41 to C20, C45 to C32, C39 to C33, C40 to C34, C44 to C35, C47 to C36, C51 to C47, C35 to C5, C48 to C51, C52 to C55, C54 to C56, C46 to C57, C49 to C58, C50 to C59, C32 to C6, C53 to C60, C30 to C7, C34 to C8, D15 to D11, D14 to D12, D17 to D16, D16 to D17, D13 to D2, D12 to D3, L9 to L10, L5 to L3, L3 to L4, L7 to L6, L6 to L7, R44 to R22, R45 to R23, R41 to R38, R42 to R39, R43 to R41, R46 to R45, R48 to R46, U10 to U4
Connections:
- net +5V: now also C21.1, U8.1 (VIN); no longer C10.2, C7.2, L2.1
- net GND: now also U3.4 (GND), C1.1, C21.2, C4.1, C63.2, R10.2, R48.2, R50.2, U1.2 (GND), U1.4 (GND), U8.2 (GND)
- net at C32.1, K1.12, L6.2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: now also C63.1
- net at C3.1: now also U1.3; no longer U3.1
- net at C5.2, L2.2: now also U3.1; no longer U3.3
- net at C12.1, C15.1, L6.1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: now also C62.2; no longer C20.2
- net at L3.1, U4.4 (RF_Out): now also C61.1; no longer C19.1
- net at D2.1 (K), D3.2 (A), U14.2 (Fterm): no longer R22.2, R23.2
- new net: C1.2, C10.2, C4.2, C7.2, L1.1, L2.1, U8.6 (VOUT)
- new net: C20.2, C62.1
- new net: C19.1, C61.2
- new net: C64.1, U3.3
- new net: C64.2, R49.1, R50.1
- new net: C9.1, R48.1, R49.2
- new net: R22.2, R23.2, U14.2 (Fterm)
- new net: C9.2, L1.2, U1.1
- new net DRIVER_EN: R10.1, U8.3 (EN/UVLO)
- no-connect marks 0 -> 2
Other:
- note added: "3dB Attenuator"
- note added: "Driver Power Switch"
- note added: "PA Driver"
- note removed: "0dBm"
- note removed: "5V"
- note removed: "6dB Attenuator"
- note removed: "PA Gain"
- moved on the sheet: C10, C12, C15, C19, C3, C32, C33, C34, C35, C36, C5, C7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

Commit message: Save unlocked Kicad files for PA Board V2
Connections:
- net at R22.2, R23.2, U14.2 (Fterm): now also D2.1 (K), D3.2 (A)
Changed lines of the file:
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@@
-    (stroke (width 0) (type default))
-  )
-  (wire (pts (xy 197.485 98.425) (xy 197.485 99.06))
     (stroke (width 0) (type default))
   )
@@
     (stroke (width 0) (type default))
   )
-  (wire (pts (xy 198.12 99.06) (xy 217.805 99.06))
-    (stroke (width 0) (type default))
-  )
   (wire (pts (xy 142.875 95.25) (xy 144.145 95.25))
     (stroke (width 0) (type default))
@@
     (stroke (width 0) (type default))
   )
+  (wire (pts (xy 197.485 99.06) (xy 217.805 99.06))
+    (stroke (width 0) (type default))
+  )
