File: electronics/bits'n_bobs/Relays/LPF_Relay/LPF_Relay.kicad_pcb (KiCad board)
At the start: 2 copper layers, 75 x 50 mm, 58 parts, among them J1 Conn_01x04, J2 Conn_01x04, J3 Conn_01x02, J4 Conn_01x03, J5 Conn_01x06, U1 MCP23017_SO, U2 ULN2003A

Commit message: Updates in electronics bits and bobs
Parts:
- F1: footprint Fuse:Fuse_0805_2012Metric -> Fuse:Fuse_Bourns_MF-SM_9.5x6.71mm
- moved C5 7.91 mm to (28.0, 9.90)
- moved L2 7.91 mm to (31.1, 9.14)
- moved C6 7.91 mm to (34.0, 9.91)
- moved D2 7.42 mm to (24.5, 11.1)
- moved F1 3.90 mm to (16.3, 8.00)
- moved R7 0.45 mm to (39.9, 29.6)
- moved R6 0.45 mm to (34.8, 29.7)
Routing:
- net GND: track 264.0 -> 247.4 mm
- net Net-(U2-COM): track 95.0 -> 87.1 mm
- net Net-(D2-K): track 8.95 -> 12.7 mm
- net Net-(J3-Pin_1): track 7.51 -> 9.77 mm
- net +3.3V: track 54.6 -> 55.8 mm
