File: electronics/bits'n_bobs/Relays/LPF_Relay/LPF_Relay.kicad_sch (KiCad schematic)
At the start: 58 parts, among them J1 Conn_01x04, J2 Conn_01x04, J3 Conn_01x02, J4 Conn_01x03, J5 Conn_01x06, U1 MCP23017_SO, U2 ULN2003A

Commit message: Updates in electronics bits and bobs
Parts:
- F1: footprint Fuse:Fuse_0805_2012Metric -> Fuse:Fuse_Bourns_MF-SM_9.5x6.71mm
Other:
- moved on the sheet: C1, C10, C11, C12, C14, C15, C2, C3, C4, C7, C9, D1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
